Commit message: add tassa example

File: examples/three/gabe_go1/urdf/go1.urdf (robot description, URDF)
Before this commit: robot go1_description, 23 links, 22 joints
Joints:
- joint RL_calf_joint: limit lower=-2.69653369433 upper=-0.916297857297 effort=33.5 velocity=28 -> lower=-2.8 upper=-0.916297857297 effort=33.5 velocity=28
